File: DIC_Board/Water_Pump.kicad_sch (KiCad schematic)
At the start: 0 parts

Commit message: Completed water pump and added the 2.7V rail
Parts:
- added C300: 100nF, Capacitor_SMD:C_0402_1005Metric, symbol Device:C
- added C301: 10uF, Capacitor_SMD:C_1206_3216Metric, symbol Device:C
- added C302: 22nF, Capacitor_SMD:C_0402_1005Metric, symbol Device:C
- added J30: 0430450200, Connector_Molex:Molex_Micro-Fit_3.0_43045-0200_2x01_P3.00mm_Horizontal, symbol Connector_Generic:Conn_01x02
- added R300: 15k, Resistor_SMD:R_0402_1005Metric, symbol Device:R
- added R301: 100k, Resistor_SMD:R_0402_1005Metric, symbol Device:R
- added R302: 1.00k, Resistor_SMD:R_0402_1005Metric, symbol Device:R
- added U30: TPS27S100APWPR, Package_SO:Texas_HTSSOP-14-1EP_4.4x5mm_P0.65mm_EP3.4x5mm_Mask3.155x3.255mm_ThermalVias, symbol DIC_Board:TPS27S100A
Connections:
- new net: C302.1, J30.1 (Pin_1), U30.5 (OUT), U30.6 (OUT), U30.7 (OUT)
- new net: R302.2, U30.13 (ILIM)
- new net: R300.2, R301.1, U30.3 (EN)
- new net +12V: C300.1, C301.1, U30.10 (IN), U30.8 (IN), U30.9 (IN)
- new net GND: C300.2, C301.2, C302.2, J30.2 (Pin_2), R301.2, R302.1, U30.12 (DIAG_EN), U30.15 (EP), U30.2 (GND)
- new net WATER_PUMP_EN: R300.1
- no-connect marks 0 -> 4
Other:
- note added: "Pump has internal reverse-polarity diode; TPS27S100A provides inductive turn-off clamp."
- note added: "SBE 5P: 10-18 V option; 1.8 A maximum turn-on surge, approximately 0.25 s."
- note added: "TPS27S100A: 40 V / 4 A smart switch; R302 = 1.00 kOhm sets approximately 2.5 A limit."

Commit message: Completed Acid Pump sheet
Other:
- moved on the sheet: C300, C301, C302, J30, R300, R301, R302
