File: DIC_Board/Water_Pump.kicad_sch (KiCad schematic)
At the start: 8 parts, among them J30 0430450200, U30 TPS27S100APWPR

Commit message: Synchronize schematic hierarchy and MCU pin map
Changed lines of the file:
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@@
 		)
 	)
-	(global_label "WATER_PUMP_EN"
+	(hierarchical_label "WATER_PUMP_EN"
 		(shape input)
 		(at 91.44 81.28 180)
-		(fields_autoplaced yes)
 		(effects
 			(font
@@
 			(justify right)
 		)
-		(property "Intersheetrefs" "${INTERSHEET_REFS}"
-			(at 72.7916 81.28 0)
-			(hide yes)
-			(show_name no)
-			(do_not_autoplace no)
-			(effects
-				(font
-					(size 1.27 1.27)
-				)
-				(justify right)
-			)
-		)
 	)

Commit message: Synchronize power, communications, and MCU configuration
Other:
- note added: "Pump has internal reverse-polarity diode TPS27S100A provides inductive turn-off clamp."
- note added: "SBE 5P: 10-18 V option 1.8 A maximum turn-on surge, approximately 0.25 s."
- note added: "TPS27S100A: 40 V / 4 A switch R302 = 1.00 kOhm sets approximately 2.5 A limit."
- note removed: "Pump has internal reverse-polarity diode; TPS27S100A provides inductive turn-off clamp."
- note removed: "SBE 5P: 10-18 V option; 1.8 A maximum turn-on surge, approximately 0.25 s."
- note removed: "TPS27S100A: 40 V / 4 A smart switch; R302 = 1.00 kOhm sets approximately 2.5 A limit."
Changed lines of the file:
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@@
 	(title_block
 		(title "Water Pump")
-		(comment 1 "Sea-Bird SBE 5P pump, 12-V high-side control")
-		(comment 2 "TPS27S100A smart switch; nominal 2.5-A current limit")
+		(comment 1 "Sea-Bird SBE 5P pump, 12V high-side control")
+		(comment 2 "TPS27S100A smart switch nominal 2.5 A current limit")
 	)
-	(text "SBE 5P: 10-18 V option; 1.8 A maximum turn-on surge, approximately 0.25 s."
+	(text "SBE 5P: 10-18 V option 1.8 A maximum turn-on surge, approximately 0.25 s."
 		(exclude_from_sim no)
 		(at 29.21 23.876 0)
@@
 		)
 	)
-	(text "Pump has internal reverse-polarity diode; TPS27S100A provides inductive turn-off clamp."
+	(text "Pump has internal reverse-polarity diode TPS27S100A provides inductive turn-off clamp."
 		(exclude_from_sim no)
 		(at 29.21 31.496 0)
@@
 		)
 	)
-	(text "TPS27S100A: 40 V / 4 A smart switch; R302 = 1.00 kOhm sets approximately 2.5 A limit."
+	(text "TPS27S100A: 40 V / 4 A switch R302 = 1.00 kOhm sets approximately 2.5 A limit."
 		(exclude_from_sim no)
 		(at 29.21 27.686 0)

Commit message: Pump fixes + doc extraction
Parts:
- removed R300: 15k, Resistor_SMD:R_0402_1005Metric, symbol Device:R
- added D4: STPS3L60U, Diode_SMD:D_SMB, symbol Device:D_Schottky
- J30: BOM Comments Pin 1 = switched +12 V; pin 2 = GND. Mating housing 0430250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 -> Pin 1 = GND; pin 2 = switched +12 V. Mating housing 0430250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
Connections:
- net GND: now also J30.1 (Pin_1), D4.2 (A); no longer J30.2 (Pin_2)
- net WATER_PUMP_EN: now also R301.1, U30.3 (EN)
- net at C302.1, U30.5 (OUT), U30.6 (OUT)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: now also J30.2 (Pin_2), D4.1 (K); no longer J30.1 (Pin_1)
Other:
- note added: "Pump has internal reverse-polarity diode; D4 and TPS27S100A provide turn-off clamping."
- note removed: "Pump has internal reverse-polarity diode TPS27S100A provides inductive turn-off clamp."
- moved on the sheet: J30, R301

Commit message: Let gpt6 astra have a go at routing. bad results.
Parts:
- U30: footprint Package_SO:Texas_HTSSOP-14-1EP_4.4x5mm_P0.65mm_EP3.4x5mm_Mask3.155x3.255mm_ThermalVias -> DIC_Board:TPS27S100_Thermal_Drill0p3
Changed lines of the file:
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@@
 			)
 		)
-		(property "Footprint" "Package_SO:Texas_HTSSOP-14-1EP_4.4x5mm_P0.65mm_EP3.4x5mm_Mask3.155x3.255mm_ThermalVias"
+		(property "Footprint" "DIC_Board:TPS27S100_Thermal_Drill0p3"
 			(at 139.7 88.9 0)
 			(hide yes)
