File: DIC_Board/mcu.kicad_sch (KiCad schematic)
At the start: 61 parts, among them J1 DM3AT-SF-PEJM5, J2 Conn_ARM_JTAG_SWD_10, SW1 SW_Push, U1 STM32L476ZGTx, U2 AB-RTCMC-32.768kHz-EOA9-S3, U3 APS6404L-3SQRX-SN, Y1 ABM8AAIG-8.000MHz-V2R-T3, Y2 ABS06-107-32.768KHZ-T

Commit message: Completed water pump and added the 2.7V rail
Connections:
- net WATER_PUMP_EN: now reaches U1.125 (PG10)
Changed lines of the file:
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@@
+		)
+	)
+	(global_label "WATER_PUMP_EN"
+		(shape output)
+		(at 290.83 104.14 180)
+		(fields_autoplaced yes)
+		(effects
+			(font
+				(size 1.27 1.27)
+			)
+			(justify right)
+		)
+		(property "Intersheetrefs" "${INTERSHEET_REFS}"
+			(at 281.94 104.14 0)
+			(hide yes)
+			(show_name no)
+			(do_not_autoplace no)
+			(effects
+				(font
+					(size 1.27 1.27)
+				)
+				(justify right)
+			)
 		)
 	)

Commit message: Separated the power sheets, did the sensor sheets.
Connections:
- net SD_CARD_DETECT_N renamed SD_DETECT_N
Other:
- moved on the sheet: C21, C23, C24, C25, C26, C27, C30, C31, FB1, J1, J2, JP1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
