File: DIC_Board/auxiliary.kicad_sch (KiCad schematic)
At the start: 15 parts, among them J12 Conn_01x04, J13 Conn_01x05_Pin, U40 MAX3226EETE, U41 TPS27S100APWPR

Commit message: Pump fixes + doc extraction
Parts:
- removed R345: 15k, Resistor_SMD:R_0402_1005Metric, symbol Device:R
Connections:
- net AUX_EN: now also R346.1, U41.3 (EN)
Changed lines of the file:
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@@
-	(wire
-		(pts
-			(xy 124.46 57.15) (xy 129.54 57.15)
-		)
-		(stroke
-			(width 0)
-			(type default)
-		)
-	)
 	(wire
 		(pts
@@
 	(wire
 		(pts
-			(xy 57.15 57.15) (xy 116.84 57.15)
+			(xy 57.15 57.15) (xy 129.54 57.15)
 		)
 		(stroke
@@
 					(unit 1)
 				)
-			)
-		)
-	)
-	(symbol
-		(lib_id "Device:R")
-		(at 120.65 57.15 90)
-		(unit 1)
-		(body_style 1)
-		(exclude_from_sim no)
-		(in_bom yes)
-		(on_board yes)
-		(in_pos_files yes)
-		(dnp no)
-		(property "Reference" "R345"
-			(at 120.904 54.356 90)
-			(show_name no)
-			(do_not_autoplace no)
-			(effects
-				(font
-					(size 1.27 1.27)
-				)
-			)
-		)
-		(property "Value" "15k"
-			(at 120.65 60.198 90)
-			(show_name no)
-			(do_not_autoplace no)
-			(effects
-				(font
-					(size 1.27 1.27)
-				)
-			)
-		)
-		(property "Footprint" "Resistor_SMD:R_0402_1005Metric"
-			(at 120.65 57.15 0)
-			(hide yes)
-			(show_name no)
-			(do_not_autoplace no)
-			(effects
-				(font
-					(size 1.27 1.27)
-				)
-			)
-		)
-		(property "Datasheet" ""
-			(at 120.65 57.15 0)
-			(hide yes)
-			(show_name no)
-			(do_not_autoplace no)
-			(effects
-				(font
-					(size 1.27 1.27)
-				)
-			)
-		)
-		(property "Description" "MCU input protection"
-			(at 120.65 57.15 0)
-			(hide yes)
-			(show_name no)
-			(do_not_autoplace no)
-			(effects
-				(font
-					(size 1.27 1.27)
-				)
-			)
-		)
-		(property "MPN" "CRCW040215K0FKED"
-			(at 120.65 57.15 0)
-			(hide yes)
-			(show_name no)
-			(do_not_autoplace no)
-			(effects
-				(font
-					(size 1.27 1.27)
-				)
-			)
-		)
-		(property "Manufacturer" "Vishay Dale"
-			(at 120.65 57.15 0)
-			(hide yes)
-			(show_name no)
-			(do_not_autoplace no)
-			(effects
-				(font
-					(size 1.27 1.27)
-				)
-			)
-		)
-		(pin "1"
-		)
-		(pin "2"
-		)
-		(instances
-			(project "DIC_Board"
-				(path "/bb0ef0df-c181-443a-843c-695cd2e0efee/973d4d17-d26b-4c44-9698-9d58019fed5c/a0b2f409-4b3d-4b66-8f84-eca7c3fb4767"
-					(reference "R345")
-					(unit 1)
-				)

Commit message: Updated board for layout! All footprints added
Parts:
- removed C335: 10uF, Capacitor_SMD:C_1206_3216Metric, symbol Device:C
- removed C340: 100nF, Capacitor_SMD:C_0402_1005Metric, symbol Device:C
- removed C343: 22nF, Capacitor_SMD:C_0402_1005Metric, symbol Device:C
- removed U41: TPS27S100APWPR, Package_SO:Texas_HTSSOP-14-1EP_4.4x5mm_P0.65mm_EP3.4x5mm_Mask3.155x3.255mm_ThermalVias, symbol DIC_Board:TPS27S100A
- added D5: BZT52C8V2-7-F, Diode_SMD:D_SOD-123, symbol Device:D_Zener
- added Q1: AO4630, Package_SO:SOIC-8_3.9x4.9mm_P1.27mm, symbol DIC_Board:AO4630_ReviewFixed
- added R345: 100k, Resistor_SMD:R_0402_1005Metric, symbol Device:R
- J12: footprint (none) -> Connector_Molex:Molex_Micro-Fit_3.0_43045-0400_2x02_P3.00mm_Horizontal; BOM Source (none) -> https://www.molex.com/en-us/products/part-detail/430450400; MPN (none) -> 0430450400; Manufacturer (none) -> Molex
- J13: footprint (none) -> DIC_Board:PinHeader_Wurth_61300511121_1x05_P2.54mm_Vertical; BOM Comments (none) -> User specified PTH male header; selected 1x5,2.54mm pitch,v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; BOM Source (none) -> https://www.we-online.com/components/products/datasheet/613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; MPN (none) -> 61300511121; Manufacturer (none) -> Wurth Elektronik
- R347: value 1.00k -> 4.7k; MPN CRCW04021K00FKED -> CRCW04024K70FKED; Manufacturer Vishay Dale -> Vishay
- U40: value MAX3226EETE -> MAX3226EETE+; symbol Interface_UART:MAX3226 -> DIC_Board:MAX3226EETE; MPN MAX3226EETE -> MAX3226EETE+
Connections:
- net +3V3: now also U40.12 (VCC); no longer U40.15 (VCC)
- net AUX_EN: now also R346.2, U40.13 (~{FORCEOFF}), U40.9 (FORCEON), Q1.2 (G1); no longer R346.1, U40.12 (FORCEON), U40.16 (~{FORCEOFF})
- net AUX_RX: now also U40.6 (R1OUT); no longer U40.9 (R1OUT)
- net AUX_TX: now also U40.8 (T1IN); no longer U40.11 (T1IN)
- net GND: now also R346.1, U40.11 (GND), U40.17 (EP), Q1.1 (S1); no longer R346.2, R347.1, U40.14 (GND)
- net at C341.1: now also U40.15 (V+); no longer U40.3 (V+)
- net at R347.2: now also Q1.7 (D1_1), Q1.8 (D1_2)
- net at C339.1: now also U40.4 (V-); no longer U40.7 (V-)
- net at J13.2 (Pin_2), J13.4 (Pin_4): now also D5.1 (K), Q1.3 (S2), R345.2
- net at J12.4 (Pin_4): now also Q1.5 (D2_1), Q1.6 (D2_2)
- net at J12.2 (Pin_2): now also U40.10 (T1OUT); no longer U40.13 (T1OUT)
- net at J12.3 (Pin_3): now also U40.5 (R1IN); no longer U40.8 (R1IN)
- net at C338.1: now also U40.2 (C2+); no longer U40.5 (C2+)
- net at C338.2: now also U40.3 (C2-); no longer U40.6 (C2-)
- net at C332.1: now also U40.16 (C1+); no longer U40.2 (C1+)
- net at C332.2: now also U40.1 (C1-); no longer U40.4 (C1-)
- new net: D5.2 (A), Q1.4 (G2), R345.1, R347.1
- no-connect marks 6 -> 2
Other:
- note added: "AUX_EN: high = load power and RS-232 TX enabled. Wait for peripheral startup before transmitting. U40 exposed pad 17 is connected to GND."
- moved on the sheet: J13
