File: DIC_Board/comms.kicad_sch (KiCad schematic)
At the start: 7 parts, among them J11 Conn_01x04, U39 MAX3226EETE

Commit message: Updated board for layout! All footprints added
Parts:
- added R348: 100k, Resistor_SMD:R_0603_1608Metric, symbol Device:R
- J11: footprint (none) -> Connector_Molex:Molex_Micro-Fit_3.0_43045-0400_2x02_P3.00mm_Horizontal; BOM Source (none) -> https://www.molex.com/en-us/products/part-detail/430450400; MPN (none) -> 0430450400; Manufacturer (none) -> Molex
- U39: value MAX3226EETE -> MAX3226EETE+; symbol Interface_UART:MAX3226 -> DIC_Board:MAX3226EETE_ReviewFixed; MPN MAX3226EETE -> MAX3226EETE+
Connections:
- net +3V3: now also U39.12 (VCC); no longer U39.15 (VCC)
- net COMM_EN: now also U39.13 (~{FORCEOFF}), U39.9 (FORCEON), R348.1; no longer U39.12 (FORCEON), U39.16 (~{FORCEOFF})
- net COMM_RX: now also U39.6 (R1OUT); no longer U39.9 (R1OUT)
- net COMM_TX: now also U39.8 (T1IN); no longer U39.11 (T1IN)
- net GND: now also U39.11 (GND), U39.17 (EP), R348.2; no longer U39.14 (GND)
- net at C331.1: now also U39.16 (C1+); no longer U39.2 (C1+)
- net at C331.2: now also U39.1 (C1-); no longer U39.4 (C1-)
- net at U39.10 (T1OUT): now also J11.2 (Pin_2)
- net at C336.1: now also U39.15 (V+); no longer U39.3 (V+)
- net at C333.1: now also U39.2 (C2+); no longer U39.5 (C2+)
- net at C333.2: now also U39.3 (C2-); no longer U39.6 (C2-)
- net at C334.1: now also U39.4 (V-); no longer U39.7 (V-)
- net at J11.3 (Pin_3): now also U39.5 (R1IN); no longer U39.8 (R1IN)
Other:
- note added: "R348 holds COMM_EN low during reset. U39 is the EETE TQFN pinout; exposed pad17 is grounded."
- moved on the sheet: J11
