File: DIC_Board/2v8.kicad_sch (KiCad schematic)
At the start: 12 parts, among them U14 TPSM53603RDAR

Commit message: Let gpt6 astra have a go at routing. bad results.
Parts:
- TP26: footprint TestPoint:TestPoint_Plated_Hole_D2.0mm -> TestPoint:TestPoint_Pad_D1.0mm
- U14: footprint Package_DFN_QFN:Texas_B3QFN-14-1EP_5x5.5mm_P0.65mm_ThermalVia -> DIC_Board:TPSM53603_Thermal_Drill0p3
Changed lines of the file:
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@@
 			)
 		)
-		(property "Footprint" "Package_DFN_QFN:Texas_B3QFN-14-1EP_5x5.5mm_P0.65mm_ThermalVia"
+		(property "Footprint" "DIC_Board:TPSM53603_Thermal_Drill0p3"
 			(at 121.92 99.06 0)
 			(hide yes)
@@
 			)
 		)
-		(property "Footprint" "TestPoint:TestPoint_Plated_Hole_D2.0mm"
+		(property "Footprint" "TestPoint:TestPoint_Pad_D1.0mm"
 			(at 217.17 95.25 0)
 			(hide yes)
