File: DIC_Board/Air_Pump.kicad_sch (KiCad schematic)
At the start: 0 parts

Commit message: Separated the power sheets, did the sensor sheets.
Parts:
- added C303: 10uF, Capacitor_SMD:C_1206_3216Metric, symbol Device:C
- added C304: 100nF, Capacitor_SMD:C_0402_1005Metric, symbol Device:C
- added C305: 22nF, Capacitor_SMD:C_0402_1005Metric, symbol Device:C
- added J33: 0430450200, Connector_Molex:Molex_Micro-Fit_3.0_43045-0200_2x01_P3.00mm_Horizontal, symbol Connector_Generic:Conn_01x02
- added R303: 15k, Resistor_SMD:R_0402_1005Metric, symbol Device:R
- added R304: 100k, Resistor_SMD:R_0402_1005Metric, symbol Device:R
- added R305: 1.00k, Resistor_SMD:R_0402_1005Metric, symbol Device:R
- added U31: TPS27S100APWPR, Package_SO:Texas_HTSSOP-14-1EP_4.4x5mm_P0.65mm_EP3.4x5mm_Mask3.155x3.255mm_ThermalVias, symbol DIC_Board:TPS27S100A
Connections:
- new net: C305.1, J33.1 (Pin_1), U31.5 (OUT), U31.6 (OUT), U31.7 (OUT)
- new net: R303.2, R304.1, U31.3 (EN)
- new net: R305.2, U31.13 (ILIM)
- new net +6V6: C303.1, C304.1, U31.10 (IN), U31.8 (IN), U31.9 (IN)
- new net AIR_PUMP_EN: R303.1
- new net GND: C303.2, C304.2, C305.2, J33.2 (Pin_2), R304.2, R305.1, U31.12 (DIAG_EN), U31.15 (EP), U31.2 (GND)
- no-connect marks 0 -> 4

Commit message: Synchronize schematic hierarchy and MCU pin map
Changed lines of the file:
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@@
 		)
 	)
-	(global_label "AIR_PUMP_EN"
+	(hierarchical_label "AIR_PUMP_EN"
 		(shape input)
 		(at 99.06 88.9 180)
-		(fields_autoplaced yes)
 		(effects
 			(font
@@
 			(justify right)
 		)
-		(property "Intersheetrefs" "${INTERSHEET_REFS}"
-			(at 83.3748 88.9 0)
-			(hide yes)
-			(show_name no)
-			(do_not_autoplace no)
-			(effects
-				(font
-					(size 1.27 1.27)
-				)
-				(justify right)
-			)
-		)
 	)

Commit message: Pump fixes + doc extraction
Parts:
- removed R303: 15k, Resistor_SMD:R_0402_1005Metric, symbol Device:R
- added D3: STPS1L40ZF, Diode_SMD:D_SOD-123F, symbol Device:D_Schottky
- J33: BOM Comments Pin 1 = switched +12 V; pin 2 = GND. Mating housing 0430250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 -> Pin 1 = GND / pump black lead; pin 2 = switched +6V6 / pump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
Connections:
- net AIR_PUMP_EN: now also R304.1, U31.3 (EN)
- net GND: now also J33.1 (Pin_1), D3.2 (A); no longer J33.2 (Pin_2)
- net at C305.1, U31.5 (OUT), U31.6 (OUT)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: now also J33.2 (Pin_2), D3.1 (K); no longer J33.1 (Pin_1)
Other:
- moved on the sheet: J33
Changed lines of the file:
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@@
+	)
+	(junction
+		(at 177.8 121.92)
+		(diameter 0)
+		(color 0 0 0 0)
 	)
 	(junction
@@
 	)
 	(junction
+		(at 167.64 91.44)
+		(diameter 0)
+		(color 0 0 0 0)
+	)
+	(junction
+		(at 177.8 91.44)
+		(diameter 0)
+		(color 0 0 0 0)
+	)
+	(junction
 		(at 152.4 121.92)
 		(diameter 0)
@@
 	(wire
 		(pts
+			(xy 177.8 91.44) (xy 191.77 91.44)
+		)
+		(stroke
+			(width 0)
+			(type default)
+		)
+	)
+	(wire
+		(pts
 			(xy 123.19 113.03) (xy 123.19 121.92)
 		)
@@
 	(wire
 		(pts
+			(xy 177.8 121.92) (xy 191.77 121.92)
+		)
+		(stroke
+			(width 0)
+			(type default)
+		)
+	)
+	(wire
+		(pts
 			(xy 167.64 113.03) (xy 167.64 121.92)
 		)
@@
 	(wire
 		(pts
-			(xy 167.64 96.52) (xy 184.15 96.52)
-		)
-		(stroke
-			(width 0)
-			(type default)
-		)
-	)
-	(wire
-		(pts
-			(xy 177.8 99.06) (xy 177.8 121.92)
-		)
-		(stroke
-			(width 0)
-			(type default)
-		)
-	)
-	(wire
-		(pts
 			(xy 147.32 81.28) (xy 147.32 76.2)
 		)
@@
 	(wire
 		(pts
+			(xy 191.77 93.98) (xy 191.77 121.92)
+		)
+		(stroke
+			(width 0)
+			(type default)
+		)
+	)
+	(wire
+		(pts
 			(xy 142.24 121.92) (xy 152.4 121.92)
 		)
@@
 	(wire
 		(pts
+			(xy 177.8 105.41) (xy 177.8 91.44)
+		)
+		(stroke
+			(width 0)
+			(type default)
+		)
+	)
+	(wire
+		(pts
 			(xy 129.54 76.2) (xy 129.54 77.47)
 		)
@@
 	(wire
 		(pts
+			(xy 167.64 91.44) (xy 177.8 91.44)
+		)
+		(stroke
+			(width 0)
+			(type default)
+		)
+	)
+	(wire
+		(pts
 			(xy 129.54 60.96) (xy 129.54 66.04)
 		)
@@
 	(wire
 		(pts
-			(xy 111.76 88.9) (xy 116.84 88.9)
-		)
-		(stroke
-			(width 0)
-			(type default)
-		)
-	)
-	(wire
-		(pts
 			(xy 142.24 76.2) (xy 152.4 76.2)
 		)
@@
 	(wire
 		(pts
+			(xy 177.8 113.03) (xy 177.8 121.92)
+		)
+		(stroke
+			(width 0)
+			(type default)
+		)
+	)
+	(wire
+		(pts
 			(xy 116.84 88.9) (xy 132.08 88.9)
 		)
@@
 	(wire
 		(pts
-			(xy 177.8 99.06) (xy 184.15 99.06)
-		)
-		(stroke
-			(width 0)
-			(type default)
-		)
-	)
-	(wire
-		(pts
 			(xy 116.84 107.95) (xy 116.84 121.92)
 		)
@@
 	(wire
 		(pts
-			(xy 99.06 88.9) (xy 104.14 88.9)
+			(xy 99.06 88.9) (xy 116.84 88.9)
 		)
 		(stroke
@@
 	)
 	(symbol
+		(lib_id "Device:D_Schottky")
+		(at 177.8 109.22 270)
+		(unit 1)
+		(body_style 1)
+		(exclude_from_sim no)
+		(in_bom yes)
+		(on_board yes)
+		(in_pos_files yes)
+		(dnp no)
+		(fields_autoplaced yes)
+		(property "Reference" "D3"
+			(at 180.34 107.6324 90)
+			(show_name no)
+			(do_not_autoplace no)
+			(effects
+				(font
+					(size 1.27 1.27)
+				)
+				(justify left)
+			)
+		)
+		(property "Value" "STPS1L40ZF"
+			(at 180.34 110.1724 90)
+			(show_name no)
+			(do_not_autoplace no)
+			(effects
+				(font
+					(size 1.27 1.27)
+				)
+				(justify left)
+			)
+		)
+		(property "Footprint" "Diode_SMD:D_SOD-123F"
+			(at 177.8 109.22 0)
+			(hide yes)
+			(show_name no)
+			(do_not_autoplace no)
+			(effects
+				(font
+					(size 1.27 1.27)
+				)
+			)
+		)
+		(property "Datasheet" "https://www.st.com/resource/en/datasheet/stps1l40.pdf"
+			(at 177.8 109.22 0)
+			(hide yes)
+			(show_name no)
+			(do_not_autoplace no)
+			(effects
+				(font
+					(size 1.27 1.27)
+				)
+			)
+		)
+		(property "Description" "40 V, 1 A low-drop Schottky freewheel rectifier, SOD-123Flat"
+			(at 177.8 109.22 0)
+			(hide yes)
+			(show_name no)
+			(do_not_autoplace no)
+			(effects
+				(font
+					(size 1.27 1.27)
+				)
+			)
+		)
+		(property "MPN" "STPS1L40ZF"
+			(at 177.8 109.22 0)
+			(hide yes)
+			(show_name no)
+			(do_not_autoplace no)
+			(effects
+				(font
+					(size 1.27 1.27)
+				)
+			)
+		)
+		(property "Manufacturer" "STMicroelectronics"
+			(at 177.8 109.22 0)
+			(hide yes)
+			(show_name no)
+			(do_not_autoplace no)
+			(effects
+				(font
+					(size 1.27 1.27)
+				)
+			)
+		)
+		(property "DigiKey" "497-16916-1-ND"
+			(at 177.8 109.22 0)
+			(hide yes)
+			(show_name no)
+			(do_not_autoplace no)
+			(effects
+				(font
+					(size 1.27 1.27)
+				)
+			)
+		)
+		(property "BOM Comments" "Freewheel clamp: pin 1 cathode to switched output; pin 2 anode to GND."
+			(at 177.8 109.22 0)
+			(hide yes)
+			(show_name no)
+			(do_not_autoplace no)
+			(effects
+				(font
+					(size 1.27 1.27)
+				)
+			)
+		)
+		(pin "1"
+		)
+		(pin "2"
+		)
+		(instances
+			(project "DIC_Board"
+				(path "/bb0ef0df-c181-443a-843c-695cd2e0efee/c0c341f0-cc08-4486-9fa7-67c0e9d2ea1a/c8a1a135-8c9f-467f-bb2b-f71123dfca54"
+					(reference "D3")
+					(unit 1)
+				)
+			)
+		)
+	)
+	(symbol
 		(lib_id "Device:C")
 		(at 134.62 69.85 0)
@@
 	(symbol
 		(lib_id "Connector_Generic:Conn_01x02")
-		(at 189.23 96.52 0)
+		(at 196.85 93.98 0)
+		(mirror x)
 		(unit 1)
 		(body_style 1)
@@
 		(dnp no)
 		(property "Reference" "J33"
-			(at 188.976 92.456 0)
+			(at 196.596 98.044 0)
 			(show_name no)
 			(do_not_autoplace no)
@@
 		)
 		(property "Value" "0430450200"
-			(at 198.882 97.79 0)
+			(at 206.502 92.71 0)
 			(show_name no)
 			(do_not_autoplace no)
@@
 		)
 		(property "Footprint" "Connector_Molex:Molex_Micro-Fit_3.0_43045-0200_2x01_P3.00mm_Horizontal"
-			(at 189.23 96.52 0)
+			(at 196.85 93.98 0)
 			(hide yes)
 			(show_name no)
@@
 		)
 		(property "Datasheet" "https://www.molex.com/content/dam/molex/molex-dot-com/products/automated/en-us/salesdrawingpdf/430/43045/430450200_sd.pdf"
-			(at 189.23 96.52 0)
+			(at 196.85 93.98 0)
 			(hide yes)
 			(show_name no)
@@
 		)
 		(property "Description" "Molex Micro-Fit 3.0 two-circuit right-angle through-hole header"
-			(at 189.23 96.52 0)
+			(at 196.85 93.98 0)
 			(hide yes)
 			(show_name no)
@@
 		)
 		(property "MPN" "0430450200"
-			(at 189.23 96.52 0)
+			(at 196.85 93.98 0)
 			(hide yes)
 			(show_name no)
@@
 		)
 		(property "Manufacturer" "Molex"
-			(at 189.23 96.52 0)
+			(at 196.85 93.98 0)
 			(hide yes)
 			(show_name no)
@@
 		)
 		(property "DigiKey" "WM1813-ND"
-			(at 189.23 96.52 0)
-			(hide yes)
-			(show_name no)
-			(do_not_autoplace no)
-			(effects
-				(font
-					(size 1.27 1.27)
-				)
-			)
-		)
-		(property "BOM Comments" "Pin 1 = switched +12 V; pin 2 = GND. Mating housing 0430250200 and female contacts required."
-			(at 189.23 96.52 0)
+			(at 196.85 93.98 0)
+			(hide yes)
+			(show_name no)
+			(do_not_autoplace no)
+			(effects
+				(font
+					(size 1.27 1.27)
+				)
+			)
+		)
+		(property "BOM Comments" "Pin 1 = GND / pump black lead; pin 2 = switched +6V6 / pump red lead. Mating housing 0430250200 and female contacts required."
+			(at 196.85 93.98 0)
 			(hide yes)
 			(show_name no)
@@
 					(unit 1)
 				)
-			)
-		)
-	)
-	(symbol
-		(lib_id "Device:R")
-		(at 107.95 88.9 90)
-		(unit 1)
-		(body_style 1)
-		(exclude_from_sim no)
-		(in_bom yes)
-		(on_board yes)
-		(in_pos_files yes)
-		(dnp no)
-		(property "Reference" "R303"
-			(at 108.204 86.106 90)
-			(show_name no)
-			(do_not_autoplace no)
-			(effects
-				(font
-					(size 1.27 1.27)
-				)
-			)
-		)
-		(property "Value" "15k"
-			(at 107.95 91.948 90)
-			(show_name no)
-			(do_not_autoplace no)
-			(effects
-				(font
-					(size 1.27 1.27)
-				)
-			)
-		)
-		(property "Footprint" "Resistor_SMD:R_0402_1005Metric"
-			(at 107.95 88.9 0)
-			(hide yes)
-			(show_name no)
-			(do_not_autoplace no)
-			(effects
-				(font
-					(size 1.27 1.27)
-				)
-			)
-		)
-		(property "Datasheet" ""
-			(at 107.95 88.9 0)
-			(hide yes)
-			(show_name no)
-			(do_not_autoplace no)
-			(effects
-				(font
-					(size 1.27 1.27)
-				)
-			)
-		)
-		(property "Description" "MCU input protection"
-			(at 107.95 88.9 0)
-			(hide yes)
-			(show_name no)
-			(do_not_autoplace no)
-			(effects
-				(font
-					(size 1.27 1.27)
-				)
-			)
-		)
-		(property "MPN" "CRCW040215K0FKED"
-			(at 107.95 88.9 0)
-			(hide yes)
-			(show_name no)
-			(do_not_autoplace no)
-			(effects
-				(font
-					(size 1.27 1.27)
-				)
-			)
-		)
-		(property "Manufacturer" "Vishay Dale"
-			(at 107.95 88.9 0)
-			(hide yes)
-			(show_name no)
-			(do_not_autoplace no)
-			(effects
-				(font
-					(size 1.27 1.27)
-				)
-			)
-		)
-		(pin "1"
-		)
-		(pin "2"
-		)
-		(instances
-			(project "DIC_Board"
-				(path "/bb0ef0df-c181-443a-843c-695cd2e0efee/c0c341f0-cc08-4486-9fa7-67c0e9d2ea1a/c8a1a135-8c9f-467f-bb2b-f71123dfca54"
-					(reference "R303")
-					(unit 1)
-				)

Commit message: Updated board for layout! All footprints added
Parts:
- J33: Design Confirmation (none) -> 2026-09-11: User confirmed the existing 6.6V supply is acce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
Other:
- moved on the sheet: J33
Changed lines of the file:
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@@
+	)
+	(junction
+		(at 177.8 91.44)
+		(diameter 0)
+		(color 0 0 0 0)
 	)
 	(junction
@@
 	)
 	(junction
-		(at 177.8 91.44)
-		(diameter 0)
-		(color 0 0 0 0)
-	)
-	(junction
 		(at 152.4 121.92)
 		(diameter 0)
@@
 	(wire
 		(pts
-			(xy 177.8 91.44) (xy 191.77 91.44)
+			(xy 177.8 91.44) (xy 194.31 91.44)
 		)
 		(stroke
@@
 	(wire
 		(pts
-			(xy 177.8 121.92) (xy 191.77 121.92)
+			(xy 177.8 121.92) (xy 194.31 121.92)
 		)
 		(stroke
@@
 	(wire
 		(pts
-			(xy 191.77 93.98) (xy 191.77 121.92)
+			(xy 194.31 93.98) (xy 194.31 121.92)
 		)
 		(stroke
@@
 	)
 	(symbol
-		(lib_id "power:+6V6")
+		(lib_id "DIC_Board:+6V6")
 		(at 129.54 60.96 0)
 		(unit 1)
@@
 	(symbol
 		(lib_id "Connector_Generic:Conn_01x02")
-		(at 196.85 93.98 0)
+		(at 199.39 93.98 0)
 		(mirror x)
 		(unit 1)
@@
 		(dnp no)
 		(property "Reference" "J33"
-			(at 196.596 98.044 0)
+			(at 199.136 98.044 0)
 			(show_name no)
 			(do_not_autoplace no)
@@
 		)
 		(property "Value" "0430450200"
-			(at 206.502 92.71 0)
+			(at 209.042 92.71 0)
 			(show_name no)
 			(do_not_autoplace no)
@@
 		)
 		(property "Footprint" "Connector_Molex:Molex_Micro-Fit_3.0_43045-0200_2x01_P3.00mm_Horizontal"
-			(at 196.85 93.98 0)
+			(at 199.39 93.98 0)
 			(hide yes)
 			(show_name no)
@@
 		)
 		(property "Datasheet" "https://www.molex.com/content/dam/molex/molex-dot-com/products/automated/en-us/salesdrawingpdf/430/43045/430450200_sd.pdf"
-			(at 196.85 93.98 0)
+			(at 199.39 93.98 0)
 			(hide yes)
 			(show_name no)
@@
 		)
 		(property "Description" "Molex Micro-Fit 3.0 two-circuit right-angle through-hole header"
-			(at 196.85 93.98 0)
+			(at 199.39 93.98 0)
 			(hide yes)
 			(show_name no)
@@
 		)
 		(property "MPN" "0430450200"
-			(at 196.85 93.98 0)
+			(at 199.39 93.98 0)
 			(hide yes)
 			(show_name no)
@@
 		)
 		(property "Manufacturer" "Molex"
-			(at 196.85 93.98 0)
+			(at 199.39 93.98 0)
 			(hide yes)
 			(show_name no)
@@
 		)
 		(property "DigiKey" "WM1813-ND"
-			(at 196.85 93.98 0)
+			(at 199.39 93.98 0)
 			(hide yes)
 			(show_name no)
@@
 		)
 		(property "BOM Comments" "Pin 1 = GND / pump black lead; pin 2 = switched +6V6 / pump red lead. Mating housing 0430250200 and female contacts required."
-			(at 196.85 93.98 0)
-			(hide yes)
-			(show_name no)
+			(at 199.39 93.98 0)
+			(hide yes)
+			(show_name no)
+			(do_not_autoplace no)
+			(effects
+				(font
+					(size 1.27 1.27)
+				)
+			)
+		)
+		(property "Design Confirmation" "2026-09-11: User confirmed the existing 6.6V supply is acceptable for the installed KNF pump. Retain 6.6V. This statement does not specify pump overload/startup limits."
+			(at 0 0 0)
+			(hide yes)
+			(show_name no)

Commit message: Let gpt6 astra have a go at routing. bad results.
Parts:
- U31: footprint Package_SO:Texas_HTSSOP-14-1EP_4.4x5mm_P0.65mm_EP3.4x5mm_Mask3.155x3.255mm_ThermalVias -> DIC_Board:TPS27S100_Thermal_Drill0p3
Changed lines of the file:
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@@
 			)
 		)
-		(property "Footprint" "Package_SO:Texas_HTSSOP-14-1EP_4.4x5mm_P0.65mm_EP3.4x5mm_Mask3.155x3.255mm_ThermalVias"
+		(property "Footprint" "DIC_Board:TPS27S100_Thermal_Drill0p3"
 			(at 147.32 96.52 0)
 			(hide yes)
