File: DIC_Board/DIC_Board.kicad_pcb (KiCad board)
At the start: 2 copper layers, 293 parts, among them J1 DM3AT-SF-PEJM5, J10 Conn_01x04, J11 Conn_01x04, J12 Conn_01x04, J13 Conn_01x05_Pin, J2 Conn_ARM_JTAG_SWD_10, J3 0430451200, J30 0430450200, J31 0430450200, J33 0430450200, J4 0430451200, J5 Conn_01x10, J6 Conn_01x04, J7 Conn_01x04, J8 Conn_01x04, J9 Conn_01x04, P1 USB4105-GF-A, Q1 AO4630, Q100 CSD18542KTTT, Q101 CSD18542KTTT, SW1 SW_Push, U1 STM32L476ZGTx, U10 TPS552882RPMR, U11 TPSM53603RDAR, U12 TPSM53603RDAR, U13 TPSM53603RDAR, U14 TPSM53603RDAR, U2 AB-RTCMC-32.768kHz-EOA9-S3, U20 DRV8823QDCARQ1, U21 DRV8823QDCARQ1, U22 DRV8823QDCARQ1, U3 APS6404L-3SQRX-SN, U30 TPS27S100APWPR, U31 TPS27S100APWPR, U32 STSPIN220, U33 TPS27S100APWPR, U34 MAX3226EETE+, U35 TPS27S100APWPR, U36 TPS27S100APWPR, U37 TPS27S100APWPR, U38 TPS27S100APWPR, U39 MAX3226EETE+, U40 MAX3226EETE+, Y1 ABM8AAIG-8.000MHz-V2R-T3, Y2 ABS06-107-32.768KHZ-T

Commit message: Let gpt6 astra have a go at routing. bad results.
Parts:
- removed the R322 at (810.0, 410.0)
- added H1: MountingHole_Pad, MountingHole:MountingHole_2.5mm_Pad, F.Cu at (24.0, 34.0)
- added H2: MountingHole_Pad, MountingHole:MountingHole_2.5mm_Pad, F.Cu at (270.0, 34.0)
- added H3: MountingHole_Pad, MountingHole:MountingHole_2.5mm_Pad, F.Cu at (270.0, 76.8)
- added H4: MountingHole_Pad, MountingHole:MountingHole_2.5mm_Pad, F.Cu at (24.0, 76.8)
- TP20, TP21, TP22, TP23, TP24, TP25, TP26: footprint TestPoint:TestPoint_Plated_Hole_D2.0mm -> TestPoint:TestPoint_Pad_D1.0mm
- U11, U12, U13, U14: footprint Package_DFN_QFN:Texas_B3QFN-14-1EP_5x5.5mm_P0.65mm_ThermalVia -> DIC_Board:TPSM53603_Thermal_Drill0p3
- U30, U31, U33, U35, U36, U37, U38: footprint Package_SO:Texas_HTSSOP-14-1EP_4.4x5mm_P0.65mm_EP3.4x5mm_Mask3.155x3.255mm_ThermalVias -> DIC_Board:TPS27S100_Thermal_Drill0p3
- moved R314 834.1 mm to (85.0, 54.0)
- moved J13 811.4 mm to (194.0, 41.9)
- moved R313 799.9 mm to (79.5, 64.5)
- moved R315 788.8 mm to (166.2, 74.3)
- moved R101 777.3 mm to (68.0, 58.3)
- moved C40 777.0 mm to (60.0, 47.1)
- moved J12 768.0 mm to (186.5, 70.7), turned to 180 degrees
- moved D5 748.0 mm to (189.0, 53.5), turned to 90 degrees
- moved R321 745.8 mm to (109.0, 64.5)
- moved R100 739.7 mm to (68.0, 56.8)
- moved C133 734.7 mm to (92.1, 53.7), turned to -90 degrees
- moved J5 724.3 mm to (90.0, 70.7), turned to 180 degrees
- moved Q101 722.8 mm to (46.0, 56.5), turned to -90 degrees
- moved C342 713.8 mm to (186.5, 64.0)
- moved R309 712.5 mm to (169.0, 59.0)
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Routing:
- net +12V: track 0.00 -> 665.2 mm, vias 0 -> 30
- net GND: track 0.00 -> 476.6 mm, vias 0 -> 268
- net /Power/12V/P_IN: track 0.00 -> 264.9 mm, vias 0 -> 5
- net /Valve Control/VALVE_SLEEP_N: track 0.00 -> 204.9 mm, vias 0 -> 8
- net /Valve Control/VALVE_LATCH: track 0.00 -> 149.0 mm, vias 0 -> 6
- net +3V3: track 0.00 -> 146.0 mm, vias 0 -> 70
- net /Valve Control/VALVE_RESET_N: track 0.00 -> 131.3 mm, vias 0 -> 8
- net /Power/6V6_EN: track 0.00 -> 104.3 mm, vias 0 -> 2
- net /Power/5V_EN: track 0.00 -> 102.1 mm, vias 0 -> 4
- net Net-(U37-EN): track 0.00 -> 100.5 mm, vias 0 -> 4
- net NRST: track 0.00 -> 98.1 mm, vias 0 -> 4
- net /STM32 MCU/RH_SDA: track 0.00 -> 92.2 mm, vias 0 -> 4
- net /Pump Control/WATER_PUMP_EN: track 0.00 -> 90.3 mm, vias 0 -> 4
- net +5V: track 0.00 -> 87.4 mm, vias 0 -> 4
- net /STM32 MCU/RH_SCL: track 0.00 -> 86.3 mm, vias 0 -> 4
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- added copper zone on In2.Cu, net +3V3
- added copper zone on In1.Cu, net GND
Other:
- board outline added: 254 x 50.8 mm
- copper layers 2 -> 4
