File: DIC_Board/DIC_Board.kicad_pcb (KiCad board)
At the start: 2 copper layers, 293 parts, among them J1 DM3AT-SF-PEJM5, J10 Conn_01x04, J11 Conn_01x04, J12 Conn_01x04, J13 Conn_01x05_Pin, J2 Conn_ARM_JTAG_SWD_10, J3 0430451200, J30 0430450200, J31 0430450200, J33 0430450200, J4 0430451200, J5 Conn_01x10, J6 Conn_01x04, J7 Conn_01x04, J8 Conn_01x04, J9 Conn_01x04, P1 USB4105-GF-A, Q1 AO4630, Q100 CSD18542KTTT, Q101 CSD18542KTTT, SW1 SW_Push, U1 STM32L476ZGTx, U10 TPS552882RPMR, U11 TPSM53603RDAR, U12 TPSM53603RDAR, U13 TPSM53603RDAR, U14 TPSM53603RDAR, U2 AB-RTCMC-32.768kHz-EOA9-S3, U20 DRV8823QDCARQ1, U21 DRV8823QDCARQ1, U22 DRV8823QDCARQ1, U3 APS6404L-3SQRX-SN, U30 TPS27S100APWPR, U31 TPS27S100APWPR, U32 STSPIN220, U33 TPS27S100APWPR, U34 MAX3226EETE+, U35 TPS27S100APWPR, U36 TPS27S100APWPR, U37 TPS27S100APWPR, U38 TPS27S100APWPR, U39 MAX3226EETE+, U40 MAX3226EETE+, Y1 ABM8AAIG-8.000MHz-V2R-T3, Y2 ABS06-107-32.768KHZ-T

Commit message: Preliminary layout
Parts:
- removed the R322 at (810.0, 410.0)
- added H1: ~, MountingHole:MountingHole_2.5mm_Pad, F.Cu at (26.5, 84.6)
- added H2: ~, MountingHole:MountingHole_2.5mm_Pad, F.Cu at (270.5, 84.6)
- added H3: ~, MountingHole:MountingHole_2.5mm_Pad, F.Cu at (270.5, 125.4)
- added H4: ~, MountingHole:MountingHole_2.5mm_Pad, F.Cu at (26.5, 125.4)
- TP20, TP21, TP22, TP23, TP24, TP25, TP26: footprint TestPoint:TestPoint_Plated_Hole_D2.0mm -> TestPoint:TestPoint_Pad_D1.0mm
- moved J13 802.3 mm to (151.5, 111.6), turned to 90 degrees
- moved C40 791.6 mm to (29.0, 120.6)
- moved J12 781.7 mm to (153.5, 89.4)
- moved R101 771.0 mm to (61.0, 107.1), turned to 90 degrees
- moved R100 749.7 mm to (42.0, 111.1), turned to 90 degrees
- moved R109 743.9 mm to (69.5, 98.6)
- moved D5 730.0 mm to (154.0, 121.6)
- moved C133 726.0 mm to (91.5, 105.6), turned to 90 degrees
- moved U12 718.9 mm to (65.5, 106.6)
- moved R4 718.8 mm to (91.5, 109.1)
- moved C342 708.7 mm to (152.5, 108.1), turned to 90 degrees
- moved R350 703.0 mm to (107.0, 124.6)
- moved Q101 700.1 mm to (53.5, 109.6)
- moved C901 697.6 mm to (76.5, 94.6), turned to 90 degrees
- moved J10 685.1 mm to (168.5, 89.4)
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Routing:
- added copper zone on In2.Cu, net +3V3
- added copper zone on In1.Cu, net GND
Other:
- board outline added: 254 x 50.8 mm
- copper layers 2 -> 4

Commit message: Changed the 12V regulator to an integrated IC
Parts:
- removed Q100, Q101: CSD18542KTTT, Package_TO_SOT_SMD:TO-263-3_TabPin2
- removed R113: 24.9k, Resistor_SMD:R_0402_1005Metric
- removed R114, R115: 1R, Resistor_SMD:R_0603_1608Metric
- C204, C214, C224: value 0.33mF -> 100uF; footprint Capacitor_THT:CP_Radial_D12.5mm_P5.00mm -> Capacitor_THT:CP_Radial_D8.0mm_P3.50mm
- R103: value 6.8m -> 10m
- U10: value TPS552882RPMR -> TPS552892RYQR; footprint DIC_Board:Texas_RPM0026A_TPS552882 -> DIC_Board:Texas_RYQ0021A_TPS552892
- moved C317 216.2 mm to (49.0, 116.1), turned to 180 degrees
- moved U36 216.0 mm to (49.0, 121.6)
- moved R314 216.0 mm to (46.5, 126.6), turned to 180 degrees
- moved R312 209.3 mm to (51.5, 126.6), turned to 180 degrees
- moved C214 207.0 mm to (36.5, 121.6), turned to 180 degrees
- moved U37 204.5 mm to (67.0, 115.6)
- moved R313 203.3 mm to (49.0, 126.6), turned to 180 degrees
- moved J4 202.5 mm to (45.0, 89.4)
- moved R316 199.8 mm to (67.0, 110.6), turned to 180 degrees
- moved R317 198.6 mm to (64.5, 110.6), turned to 180 degrees
- moved C319 197.3 mm to (52.2, 116.3), turned to 90 degrees
- moved R315 197.3 mm to (70.8, 111.6), turned to -90 degrees
- moved J3 192.8 mm to (31.1, 112.1), turned to 90 degrees
- moved C327 192.0 mm to (72.2, 111.6), turned to 90 degrees
- moved C204 190.8 mm to (37.2, 87.6), turned to 180 degrees
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Connections:
- net Net-(U10-FB) renamed /Power/12V/FB_12V
- C102 pad 1: Net-(Q100-S) -> Net-(U10-SW1)
- C103 pad 1: Net-(U10-BOOT2) -> Net-(U10-SW2)
- C103 pad 2: Net-(C103-Pad2) -> Net-(U10-BOOT2)
- C105 pad 1: Net-(U10-COMP) -> /Power/12V/COMP_12V
- C106 pad 1: Net-(U10-VCC) -> /Power/12V/VCC_BIAS
- C109 pad 1: Net-(U10-ISP) -> /Power/12V/VOUT_RAW
- C110 pad 1: Net-(U10-ISP) -> /Power/12V/VOUT_RAW
- C111 pad 1: Net-(U10-ISP) -> /Power/12V/VOUT_RAW
- C112 pad 1: Net-(U10-ISP) -> /Power/12V/VOUT_RAW
- C113 pad 1: Net-(U10-ISP) -> /Power/12V/VOUT_RAW
- C119 pad 1: Net-(U10-DITH/SYNC) -> /Power/12V/DITHER
- C40 pad 1: Net-(U10-ISP) -> /Power/12V/VOUT_RAW
- L10 pad 1: Net-(Q100-S) -> Net-(U10-SW1)
- L10 pad 2: Net-(C103-Pad2) -> Net-(U10-SW2)
- R100 pad 2: Net-(U10-EN/UVLO) -> /Power/12V/EN_UVLO
- R101 pad 1: GND -> /Power/12V/EN_UVLO
- R101 pad 2: Net-(U10-EN/UVLO) -> GND
- R102 pad 1: Net-(U10-FSW) -> /Power/12V/FSW_SET
- R103 pad 1: Net-(U10-ISP) -> /Power/12V/VOUT_RAW
- R106 pad 1: Net-(C104-Pad1) -> /Power/12V/COMP_12V
- R106 pad 2: Net-(U10-COMP) -> Net-(C104-Pad1)
- R112 pad 1: Net-(U10-MODE) -> /Power/12V/MODE_SEL
- U10 pad 1: Net-(U10-DR1L) -> /Power/12V/EN_UVLO
- U10 pad 10: GND -> Net-(U10-SW2)
- U10 pad 11: Net-(U10-ISP) -> /Power/12V/VOUT_RAW
- U10 pad 12: Net-(U10-ISP) -> /Power/12V/VOUT_RAW
- U10 pad 15: Net-(U10-MODE) -> /Power/12V/COMP_12V
- U10 pad 17: Net-(U10-ILIM) -> GND
- U10 pad 18: Net-(U10-COMP) -> /Power/12V/VCC_BIAS
- U10 pad 19: Net-(U10-VCC) -> Net-(U10-BOOT2)
- U10 pad 2: Net-(U10-DR1H) -> /Power/12V/MODE_SEL
- U10 pad 20: Net-(U10-BOOT2) -> Net-(U10-BOOT1)
- U10 pad 21: Net-(C103-Pad2) -> unconnected-(U10-EXTVCC-Pad21)
- U10 pad 3: /Power/12V/P_IN -> unconnected-(U10-PG-Pad3)
- U10 pad 4: Net-(U10-EN/UVLO) -> unconnected-(U10-CC-Pad4)
- U10 pad 5: unconnected-(U10-PG-Pad5) -> /Power/12V/DITHER
- U10 pad 6: unconnected-(U10-CC-Pad6) -> /Power/12V/FSW_SET
- U10 pad 7: Net-(U10-DITH/SYNC) -> /Power/12V/P_IN
- U10 pad 8: Net-(U10-FSW) -> Net-(U10-SW1)
Other:
- outline, holes or cut-outs redrawn

Commit message: minor PCB
Parts:
- moved J5 11.0 mm to (74.5, 89.4)
- moved D1 0.50 mm to (259.0, 94.1)
Other:
- outline, holes or cut-outs redrawn
Changed lines of the file:
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@@
 	)
 	(footprint "Capacitor_SMD:CP_Elec_8x10.5"
+		(locked yes)
 		(layer "F.Cu")
 		(at 131.5 87.1)
@@
 	(footprint "Connector_Molex:Molex_Micro-Fit_3.0_43045-1000_2x05_P3.00mm_Horizontal"
 		(layer "F.Cu")
-		(at 85.5 89.399999)
+		(at 74.5 89.399999)
 		(descr "Molex Micro-Fit 3.0 Connector System, 43045-1000 (alternative finishes: 43045-100x), 5 Pins per row (https://www.molex.com/pdm_docs/sd/430450201_sd.pdf)")
 		(tags "connector Molex Micro-Fit_3.0 horizontal")
@@
 	(footprint "Package_TO_SOT_SMD:SOT-523"
 		(layer "F.Cu")
-		(at 258.5 94.1 90)
+		(at 259 94.1 90)
 		(descr "SOT523, https://www.diodes.com/assets/Package-Files/SOT523.pdf")
 		(tags "SOT-523")
@@
 	(gr_line
 		(start 21.5 79.6)
-		(end 224.925 79.6)
+		(end 223 79.6)
 		(stroke
 			(width 0.05)
@@
 	)
 	(gr_line
-		(start 224.925 79.6)
-		(end 226.925 83.6)
+		(start 223 79.6)
+		(end 225 84.6)
 		(stroke
 			(width 0.05)
@@
 	)
 	(gr_line
-		(start 226.925 83.6)
-		(end 230.925 83.6)
+		(start 225 84.6)
+		(end 232.5 84.6)
 		(stroke
 			(width 0.05)
@@
 	)
 	(gr_line
-		(start 230.925 83.6)
-		(end 232.925 79.6)
+		(start 232.5 84.6)
+		(end 235 79.6)
 		(stroke
 			(width 0.05)
@@
 	)
 	(gr_line
-		(start 232.925 79.6)
+		(start 235 79.6)
 		(end 275.5 79.6)
 		(stroke

Commit message: resized the board to 9.5 in by 2 in
Parts:
- moved C224 50.8 mm to (39.3, 98.6)
- moved C127 30.8 mm to (136.5, 107.8)
- moved C126 26.6 mm to (125.8, 125.8)
- moved C330 24.0 mm to (157.0, 112.1)
- moved C328 23.7 mm to (168.0, 98.3)
- moved R324 23.2 mm to (188.2, 122.1)
- moved R327 22.0 mm to (190.0, 125.3)
- moved J30 21.8 mm to (182.0, 106.3)
- moved C324 20.6 mm to (190.0, 122.1)
- moved C334 20.0 mm to (163.5, 80.8)
- moved C300 17.4 mm to (176.8, 115.1)
- moved J33 17.4 mm to (190.5, 103.6)
- moved C342 17.3 mm to (176.0, 95.1)
- moved R343 16.9 mm to (189.2, 119.6)
- moved R310 16.6 mm to (169.8, 95.8)
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Other:
- board size 254 x 50.8 mm -> 241.3 x 50.8 mm
