File: DIC_Board/DIC_Board.kicad_sch (KiCad schematic)
At the start: 0 parts

Commit message: Let gpt6 astra have a go at routing. bad results.
Parts:
- added H1, H2, H3, H4: MountingHole_Pad, MountingHole:MountingHole_2.5mm_Pad, symbol Mechanical:MountingHole_Pad
Connections:
- new net GND: H1.1, H2.1, H3.1, H4.1
