File: DIC_Board/Licor.kicad_sch (KiCad schematic)
At the start: 14 parts, among them J35 0430450400, U33 TPS27S100APWPR, U34 MAX3226EETE

Commit message: Synchronize schematic hierarchy and MCU pin map
Parts:
- removed J35: 0430450400, Connector_Molex:Molex_Micro-Fit_3.0_43045-0400_2x02_P3.00mm_Horizontal, symbol Connector_Generic:Conn_02x02_Odd_Even
- added J10: Conn_01x04, symbol Connector_Generic:Conn_01x04
Connections:
- net GND: now also J10.1 (Pin_1)
- net at U34.13 (T1OUT): now also J10.2 (Pin_2)
- net at U34.8 (R1IN): now also J10.3 (Pin_3)
- net at C308.1, U33.5 (OUT), U33.6 (OUT)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: now also J10.4 (Pin_4)

Commit message: Pump fixes + doc extraction
Parts:
- removed R306: 15k, Resistor_SMD:R_0402_1005Metric, symbol Device:R
Connections:
- net LICOR_EN: now also R307.1, U33.3 (EN)
Changed lines of the file:
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@@
-	(wire
-		(pts
-			(xy 115.57 52.07) (xy 120.65 52.07)
-		)
-		(stroke
-			(width 0)
-			(type default)
-		)
-	)
 	(wire
 		(pts
@@
 	(wire
 		(pts
-			(xy 48.26 52.07) (xy 107.95 52.07)
+			(xy 48.26 52.07) (xy 120.65 52.07)
 		)
 		(stroke
@@
 					(unit 1)
 				)
-			)
-		)
-	)
-	(symbol
-		(lib_id "Device:R")
-		(at 111.76 52.07 90)
-		(unit 1)
-		(body_style 1)
-		(exclude_from_sim no)
-		(in_bom yes)
-		(on_board yes)
-		(in_pos_files yes)
-		(dnp no)
-		(property "Reference" "R306"
-			(at 112.014 49.276 90)
-			(show_name no)
-			(do_not_autoplace no)
-			(effects
-				(font
-					(size 1.27 1.27)
-				)
-			)
-		)
-		(property "Value" "15k"
-			(at 111.76 55.118 90)
-			(show_name no)
-			(do_not_autoplace no)
-			(effects
-				(font
-					(size 1.27 1.27)
-				)
-			)
-		)
-		(property "Footprint" "Resistor_SMD:R_0402_1005Metric"
-			(at 111.76 52.07 0)
-			(hide yes)
-			(show_name no)
-			(do_not_autoplace no)
-			(effects
-				(font
-					(size 1.27 1.27)
-				)
-			)
-		)
-		(property "Datasheet" ""
-			(at 111.76 52.07 0)
-			(hide yes)
-			(show_name no)
-			(do_not_autoplace no)
-			(effects
-				(font
-					(size 1.27 1.27)
-				)
-			)
-		)
-		(property "Description" "MCU input protection"
-			(at 111.76 52.07 0)
-			(hide yes)
-			(show_name no)
-			(do_not_autoplace no)
-			(effects
-				(font
-					(size 1.27 1.27)
-				)
-			)
-		)
-		(property "MPN" "CRCW040215K0FKED"
-			(at 111.76 52.07 0)
-			(hide yes)
-			(show_name no)
-			(do_not_autoplace no)
-			(effects
-				(font
-					(size 1.27 1.27)
-				)
-			)
-		)
-		(property "Manufacturer" "Vishay Dale"
-			(at 111.76 52.07 0)
-			(hide yes)
-			(show_name no)
-			(do_not_autoplace no)
-			(effects
-				(font
-					(size 1.27 1.27)
-				)
-			)
-		)
-		(pin "1"
-		)
-		(pin "2"
-		)
-		(instances
-			(project "DIC_Board"
-				(path "/bb0ef0df-c181-443a-843c-695cd2e0efee/15388a04-aea8-414b-8903-58a719a8054d/90896a52-6a15-4861-9fbc-84f5783b3f4c"
-					(reference "R306")
-					(unit 1)
-				)

Commit message: Updated board for layout! All footprints added
Parts:
- J10: footprint (none) -> Connector_Molex:Molex_Micro-Fit_3.0_43045-0400_2x02_P3.00mm_Horizontal; BOM Source (none) -> https://www.molex.com/en-us/products/part-detail/430450400; Design Confirmation (none) -> 2026-09-11: User accepted the existing nominal 12V supply f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; MPN (none) -> 0430450400; Manufacturer (none) -> Molex
- U34: value MAX3226EETE -> MAX3226EETE+; symbol Interface_UART:MAX3226 -> DIC_Board:MAX3226EETE_ReviewFixed; MPN MAX3226EETE -> MAX3226EETE+
Connections:
- net +3V3: now also U34.12 (VCC); no longer U34.15 (VCC)
- net GND: now also U34.11 (GND), U34.17 (EP); no longer U34.14 (GND)
- net LICOR_EN: now also U34.13 (~{FORCEOFF}), U34.9 (FORCEON); no longer U34.12 (FORCEON), U34.16 (~{FORCEOFF})
- net LICOR_RX: now also U34.6 (R1OUT); no longer U34.9 (R1OUT)
- net LICOR_TX: now also U34.8 (T1IN); no longer U34.11 (T1IN)
- net at J10.2 (Pin_2): now also U34.10 (T1OUT); no longer U34.13 (T1OUT)
- net at J10.3 (Pin_3): now also U34.5 (R1IN); no longer U34.8 (R1IN)
- net at U34.1 (C1-): now also C309.2
- net at C309.1: now also U34.16 (C1+); no longer U34.2 (C1+)
- net at C311.1: now also U34.15 (V+); no longer U34.3 (V+)
- net at U34.4 (V-): now also C312.1; no longer C309.2
- net at C310.1: now also U34.2 (C2+); no longer U34.5 (C2+)
- net at C310.2: now also U34.3 (C2-); no longer U34.6 (C2-)
- net at U34.7 (~{INVALID}): no longer C312.1
Changed lines of the file:
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@@
-	)
-	(junction
-		(at 83.82 144.78)
-		(diameter 0)
-		(color 0 0 0 0)
 	)
 	(junction
@@
 		(pts
 			(xy 156.21 74.93) (xy 156.21 85.09)
-		)
-		(stroke
-			(width 0)
-			(type default)
-		)
-	)
-	(wire
-		(pts
-			(xy 83.82 144.78) (xy 85.09 144.78)
 		)
 		(stroke
@@
 			)
 		)
-		(property "Footprint" ""
+		(property "Footprint" "Connector_Molex:Molex_Micro-Fit_3.0_43045-0400_2x02_P3.00mm_Horizontal"
 			(at 224.79 87.63 0)
 			(hide yes)
@@
 		(property "Description" "Generic connector, single row, 01x04, script generated (kicad-library-utils/schlib/autogen/connector/)"
 			(at 224.79 87.63 0)
+			(hide yes)
+			(show_name no)
+			(do_not_autoplace no)
+			(effects
+				(font
+					(size 1.27 1.27)
+				)
+			)
+		)
+		(property "BOM Source" "https://www.molex.com/en-us/products/part-detail/430450400"
+			(at 0 0 0)
+			(hide yes)
+			(show_name no)
+			(do_not_autoplace no)
+			(effects
+				(font
+					(size 1.27 1.27)
+				)
+			)
+		)
+		(property "Manufacturer" "Molex"
+			(at 0 0 0)
+			(hide yes)
+			(show_name no)
+			(do_not_autoplace no)
+			(effects
+				(font
+					(size 1.27 1.27)
+				)
+			)
+		)
+		(property "MPN" "0430450400"
+			(at 0 0 0)
+			(hide yes)
+			(show_name no)
+			(do_not_autoplace no)
+			(effects
+				(font
+					(size 1.27 1.27)
+				)
+			)
+		)
+		(property "Design Confirmation" "2026-09-11: User accepted the existing nominal 12V supply for LI-830; retain present supply and interface."
+			(at 0 0 0)
 			(hide yes)
 			(show_name no)
@@
 	)
 	(symbol
-		(lib_id "Interface_UART:MAX3226")
+		(lib_id "DIC_Board:MAX3226EETE_ReviewFixed")
 		(at 104.14 142.24 0)
 		(unit 1)
@@
 			)
 		)
-		(property "Value" "MAX3226EETE"
+		(property "Value" "MAX3226EETE+"
 			(at 104.14 128.016 0)
 			(show_name no)
@@
 			)
 		)
-		(property "Datasheet" "https://datasheets.maximintegrated.com/en/ds/MAX3224-MAX3245.pdf"
+		(property "Datasheet" "https://www.analog.com/media/en/technical-documentation/data-sheets/MAX3224E-MAX3245E.pdf"
 			(at 104.14 144.78 0)
 			(hide yes)
@@
 			)
 		)
-		(property "MPN" "MAX3226EETE"
+		(property "MPN" "MAX3226EETE+"
 			(at 104.14 142.24 0)
 			(hide yes)
@@
 			)
 		)
+		(pin "14"
+		)
+		(pin "16"
+		)
+		(pin "15"
+		)
 		(pin "1"
 		)
@@
 		(pin "13"
 		)
-		(pin "14"
-		)
-		(pin "15"
-		)
-		(pin "16"
+		(pin "17"
 		)
 		(instances

Commit message: Let gpt6 astra have a go at routing. bad results.
Parts:
- U33: footprint Package_SO:Texas_HTSSOP-14-1EP_4.4x5mm_P0.65mm_EP3.4x5mm_Mask3.155x3.255mm_ThermalVias -> DIC_Board:TPS27S100_Thermal_Drill0p3
Changed lines of the file:
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@@
 			)
 		)
-		(property "Footprint" "Package_SO:Texas_HTSSOP-14-1EP_4.4x5mm_P0.65mm_EP3.4x5mm_Mask3.155x3.255mm_ThermalVias"
+		(property "Footprint" "DIC_Board:TPS27S100_Thermal_Drill0p3"
 			(at 151.13 59.69 0)
 			(hide yes)
