File: DIC_Board/actuators.kicad_sch (KiCad schematic)
At the start: 0 parts

Commit message: Wrapping up schematic
Parts:
- added C317, C325: 10uF, Capacitor_SMD:C_1206_3216Metric, symbol Device:C
- added C318, C326: 100nF, Capacitor_SMD:C_0402_1005Metric, symbol Device:C
- added C319, C327: 22nF, Capacitor_SMD:C_0402_1005Metric, symbol Device:C
- added J5: Conn_01x10, symbol Connector_Generic:Conn_01x10
- added R312, R315: 15k, Resistor_SMD:R_0402_1005Metric, symbol Device:R
- added R313, R316: 100k, Resistor_SMD:R_0402_1005Metric, symbol Device:R
- added R314, R317: 1.00k, Resistor_SMD:R_0402_1005Metric, symbol Device:R
- added U36, U37: TPS27S100APWPR, Package_SO:Texas_HTSSOP-14-1EP_4.4x5mm_P0.65mm_EP3.4x5mm_Mask3.155x3.255mm_ThermalVias, symbol DIC_Board:TPS27S100A
Connections:
- new net: R314.2, U36.13 (ILIM)
- new net: R312.2, R313.1, U36.3 (EN)
- new net: C319.1, J5.2 (Pin_2), U36.5 (OUT), U36.6 (OUT), U36.7 (OUT)
- new net: R317.2, U37.13 (ILIM)
- new net: R315.2, R316.1, U37.3 (EN)
- new net: C327.1, J5.7 (Pin_7), U37.5 (OUT), U37.6 (OUT), U37.7 (OUT)
- new net +12V: C317.1, C318.1, C325.1, C326.1, U36.10 (IN), U36.8 (IN), U36.9 (IN), U37.10 (IN), U37.8 (IN), U37.9 (IN)
- new net ACTUATOR_1_CURRENT: J5.5 (Pin_5)
- new net ACTUATOR_1_EN: R312.1
- new net ACTUATOR_1_POS: J5.4 (Pin_4)
- new net ACTUATOR_1_PWM: J5.3 (Pin_3)
- new net ACTUATOR_2_CURRENT: J5.10 (Pin_10)
- new net ACTUATOR_2_EN: R315.1
- new net ACTUATOR_2_POS: J5.9 (Pin_9)
- new net ACTUATOR_2_PWM: J5.8 (Pin_8)
- new net GND: C317.2, C318.2, C319.2, C325.2, C326.2, C327.2, J5.1 (Pin_1), J5.6 (Pin_6), R313.2, R314.1, R316.2, R317.1, U36.12 (DIAG_EN), U36.15 (EP), U36.2 (GND), U37.12 (DIAG_EN), U37.15 (EP), U37.2 (GND)
- no-connect marks 0 -> 8

Commit message: Synchronize schematic hierarchy and MCU pin map
Changed lines of the file:
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@@
 		)
 	)
-	(global_label "ACTUATOR_1_POS"
+	(hierarchical_label "ACTUATOR_1_POS"
 		(shape output)
 		(at 251.46 93.98 180)
-		(fields_autoplaced yes)
 		(effects
 			(font
@@
 			(justify right)
 		)
-		(property "Intersheetrefs" "${INTERSHEET_REFS}"
-			(at 232.2067 93.98 0)
-			(hide yes)
-			(show_name no)
-			(do_not_autoplace no)
-			(effects
-				(font
-					(size 1.27 1.27)
-				)
-				(justify right)
-			)
-		)
 	)
-	(global_label "ACTUATOR_1_PWM"
+	(hierarchical_label "ACTUATOR_1_PWM"
 		(shape input)
 		(at 251.46 91.44 180)
-		(fields_autoplaced yes)
 		(effects
 			(font
@@
 			(justify right)
 		)
-		(property "Intersheetrefs" "${INTERSHEET_REFS}"
-			(at 231.8439 91.44 0)
-			(hide yes)
-			(show_name no)
-			(do_not_autoplace no)
-			(effects
-				(font
-					(size 1.27 1.27)
-				)
-				(justify right)
-			)
-		)
 	)
-	(global_label "ACTUATOR_2_EN"
+	(hierarchical_label "ACTUATOR_2_EN"
 		(shape input)
 		(at 44.45 140.97 180)
-		(fields_autoplaced yes)
 		(effects
 			(font
@@
 			(justify right)
 		)
-		(property "Intersheetrefs" "${INTERSHEET_REFS}"
-			(at 26.5272 140.97 0)
-			(hide yes)
-			(show_name no)
-			(do_not_autoplace no)
-			(effects
-				(font
-					(size 1.27 1.27)
-				)
-				(justify right)
-			)
-		)
 	)
-	(global_label "ACTUATOR_1_EN"
+	(hierarchical_label "ACTUATOR_1_EN"
 		(shape input)
 		(at 44.45 53.34 180)
-		(fields_autoplaced yes)
 		(effects
 			(font
@@
 			(justify right)
 		)
-		(property "Intersheetrefs" "${INTERSHEET_REFS}"
-			(at 25.8016 53.34 0)
-			(hide yes)
-			(show_name no)
-			(do_not_autoplace no)
-			(effects
-				(font
-					(size 1.27 1.27)
-				)
-				(justify right)
-			)
-		)
 	)
-	(global_label "ACTUATOR_1_CURRENT"
+	(hierarchical_label "ACTUATOR_1_CURRENT"
 		(shape output)
 		(at 251.46 96.52 180)
-		(fields_autoplaced yes)
 		(effects
 			(font
@@
 			(justify right)
 		)
-		(property "Intersheetrefs" "${INTERSHEET_REFS}"
-			(at 227.4291 96.52 0)
-			(hide yes)
-			(show_name no)
-			(do_not_autoplace no)
-			(effects
-				(font
-					(size 1.27 1.27)
-				)
-				(justify right)
-			)
-		)
 	)
-	(global_label "ACTUATOR_2_CURRENT"
+	(hierarchical_label "ACTUATOR_2_CURRENT"
 		(shape output)
 		(at 251.46 109.22 180)
-		(fields_autoplaced yes)
 		(effects
 			(font
@@
 			(justify right)
 		)
-		(property "Intersheetrefs" "${INTERSHEET_REFS}"
-			(at 227.4291 109.22 0)
-			(hide yes)
-			(show_name no)
-			(do_not_autoplace no)
-			(effects
-				(font
-					(size 1.27 1.27)
-				)
-				(justify right)
-			)
-		)
 	)
-	(global_label "ACTUATOR_2_PWM"
+	(hierarchical_label "ACTUATOR_2_PWM"
 		(shape input)
 		(at 251.46 104.14 180)
-		(fields_autoplaced yes)
 		(effects
 			(font
@@
 			(justify right)
 		)
-		(property "Intersheetrefs" "${INTERSHEET_REFS}"
-			(at 231.8439 104.14 0)
-			(hide yes)
-			(show_name no)
-			(do_not_autoplace no)
-			(effects
-				(font
-					(size 1.27 1.27)
-				)
-				(justify right)
-			)
-		)
 	)
-	(global_label "ACTUATOR_2_POS"
+	(hierarchical_label "ACTUATOR_2_POS"
 		(shape output)
 		(at 251.46 106.68 180)
-		(fields_autoplaced yes)
 		(effects
 			(font
@@
 			(justify right)
 		)
-		(property "Intersheetrefs" "${INTERSHEET_REFS}"
-			(at 232.2067 106.68 0)
-			(hide yes)
-			(show_name no)
-			(do_not_autoplace no)
-			(effects
-				(font
-					(size 1.27 1.27)
-				)
-				(justify right)
-			)
-		)
 	)

Commit message: Updated board for layout! All footprints added
Parts:
- J5: footprint (none) -> Connector_Molex:Molex_Micro-Fit_3.0_43045-1000_2x05_P3.00mm_Horizontal; BOM Source (none) -> https://www.molex.com/en-us/products/part-detail/430451000; Design Confirmation (none) -> 2026-09-11: User confirmed the existing actuator/controller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; MPN (none) -> 0430451000; Manufacturer (none) -> Molex
Changed lines of the file:
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@@
 			)
 		)
-		(property "Footprint" ""
+		(property "Footprint" "Connector_Molex:Molex_Micro-Fit_3.0_43045-1000_2x05_P3.00mm_Horizontal"
 			(at 261.62 96.52 0)
 			(hide yes)
@@
 			(hide yes)
 			(show_name no)
+			(do_not_autoplace no)
+			(effects
+				(font
+					(size 1.27 1.27)
+				)
+			)
+		)
+		(property "Design Confirmation" "2026-09-11: User confirmed the existing actuator/controller interface is acceptable; retain the implemented interface."
+			(at 0 0 0)
+			(hide yes)
+			(show_name no)
+			(do_not_autoplace no)
+			(effects
+				(font
+					(size 1.27 1.27)
+				)
+			)
+		)
+		(property "MPN" "0430451000"
+			(at 0 0 0)
+			(hide yes)
+			(show_name no)
+			(do_not_autoplace no)
+			(effects
+				(font
+					(size 1.27 1.27)
+				)
+			)
+		)
+		(property "Manufacturer" "Molex"
+			(at 0 0 0)
+			(hide yes)
+			(show_name no)
+			(do_not_autoplace no)
+			(effects
+				(font
+					(size 1.27 1.27)
+				)
+			)
+		)
+		(property "BOM Source" "https://www.molex.com/en-us/products/part-detail/430451000"
+			(at 0 0 0)
+			(hide yes)
+			(show_name no)

Commit message: Let gpt6 astra have a go at routing. bad results.
Parts:
- U36, U37: footprint Package_SO:Texas_HTSSOP-14-1EP_4.4x5mm_P0.65mm_EP3.4x5mm_Mask3.155x3.255mm_ThermalVias -> DIC_Board:TPS27S100_Thermal_Drill0p3
Changed lines of the file:
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@@
 			)
 		)
-		(property "Footprint" "Package_SO:Texas_HTSSOP-14-1EP_4.4x5mm_P0.65mm_EP3.4x5mm_Mask3.155x3.255mm_ThermalVias"
+		(property "Footprint" "DIC_Board:TPS27S100_Thermal_Drill0p3"
 			(at 92.71 60.96 0)
 			(hide yes)
@@
 			)
 		)
-		(property "Footprint" "Package_SO:Texas_HTSSOP-14-1EP_4.4x5mm_P0.65mm_EP3.4x5mm_Mask3.155x3.255mm_ThermalVias"
+		(property "Footprint" "DIC_Board:TPS27S100_Thermal_Drill0p3"
 			(at 92.71 148.59 0)
 			(hide yes)
