File: DIC_Board/o2_sensor.kicad_sch (KiCad schematic)
At the start: 0 parts

Commit message: Wrapping up schematic
Parts:
- added C328: 10uF, Capacitor_SMD:C_1206_3216Metric, symbol Device:C
- added C329: 100nF, Capacitor_SMD:C_0402_1005Metric, symbol Device:C
- added C330: 22nF, Capacitor_SMD:C_0402_1005Metric, symbol Device:C
- added J7: Conn_01x04, symbol Connector_Generic:Conn_01x04
- added R340: 15k, Resistor_SMD:R_0402_1005Metric, symbol Device:R
- added R341: 100k, Resistor_SMD:R_0402_1005Metric, symbol Device:R
- added R342: 1.00k, Resistor_SMD:R_0402_1005Metric, symbol Device:R
- added U38: TPS27S100APWPR, Package_SO:Texas_HTSSOP-14-1EP_4.4x5mm_P0.65mm_EP3.4x5mm_Mask3.155x3.255mm_ThermalVias, symbol DIC_Board:TPS27S100A
Connections:
- new net: R340.2, R341.1, U38.3 (EN)
- new net: R342.2, U38.13 (ILIM)
- new net: C330.1, J7.4 (Pin_4), U38.5 (OUT), U38.6 (OUT), U38.7 (OUT)
- new net +5V: C328.1, C329.1, U38.10 (IN), U38.8 (IN), U38.9 (IN)
- new net GND: C328.2, C329.2, C330.2, J7.1 (Pin_1), R341.2, R342.1, U38.12 (DIAG_EN), U38.15 (EP), U38.2 (GND)
- new net O2_SENSOR_EN: R340.1
- new net O2_SENSOR_RX: J7.3 (Pin_3)
- new net O2_SENSOR_TX: J7.2 (Pin_2)
- no-connect marks 0 -> 4

Commit message: Synchronize schematic hierarchy and MCU pin map
Changed lines of the file:
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@@
 	(wire
 		(pts
-			(xy 186.69 115.57) (xy 189.23 115.57)
-		)
-		(stroke
-			(width 0)
-			(type default)
-		)
-	)
-	(wire
-		(pts
-			(xy 186.69 118.11) (xy 191.77 118.11)
+			(xy 189.23 109.22) (xy 193.04 109.22)
 		)
 		(stroke
@@
 	(wire
 		(pts
-			(xy 171.45 111.76) (xy 193.04 111.76)
+			(xy 166.37 111.76) (xy 193.04 111.76)
 		)
 		(stroke
@@
 	(wire
 		(pts
-			(xy 171.45 101.6) (xy 171.45 111.76)
+			(xy 166.37 101.6) (xy 166.37 111.76)
 		)
 		(stroke
@@
 	(wire
 		(pts
-			(xy 154.94 101.6) (xy 171.45 101.6)
+			(xy 154.94 101.6) (xy 166.37 101.6)
 		)
 		(stroke
@@
 	(wire
 		(pts
-			(xy 189.23 115.57) (xy 189.23 106.68)
-		)
-		(stroke
-			(width 0)
-			(type default)
-		)
-	)
-	(wire
-		(pts
 			(xy 154.94 118.11) (xy 154.94 127)
 		)
@@
 	(wire
 		(pts
-			(xy 191.77 118.11) (xy 191.77 109.22)
-		)
-		(stroke
-			(width 0)
-			(type default)
-		)
-	)
-	(wire
-		(pts
 			(xy 139.7 116.84) (xy 139.7 127)
 		)
@@
 	(wire
 		(pts
-			(xy 191.77 109.22) (xy 193.04 109.22)
-		)
-		(stroke
-			(width 0)
-			(type default)
-		)
-	)
-	(wire
-		(pts
 			(xy 134.62 86.36) (xy 134.62 81.28)
 		)
@@
 		)
 	)
-	(global_label "O2_SENSOR_TX"
+	(hierarchical_label "O2_SENSOR_TX"
 		(shape input)
-		(at 186.69 115.57 180)
-		(fields_autoplaced yes)
+		(at 189.23 106.68 180)
 		(effects
 			(font
@@
 			(justify right)
 		)
-		(property "Intersheetrefs" "${INTERSHEET_REFS}"
-			(at 169.5535 115.57 0)
-			(hide yes)
-			(show_name no)
-			(do_not_autoplace no)
-			(effects
-				(font
-					(size 1.27 1.27)
-				)
-				(justify right)
-			)
-		)
-	)
-	(global_label "O2_SENSOR_EN"
+	)
+	(hierarchical_label "O2_SENSOR_EN"
 		(shape input)
 		(at 86.36 93.98 180)
-		(fields_autoplaced yes)
 		(effects
 			(font
@@
 			(justify right)
 		)
-		(property "Intersheetrefs" "${INTERSHEET_REFS}"
-			(at 68.9211 93.98 0)
-			(hide yes)
-			(show_name no)
-			(do_not_autoplace no)
-			(effects
-				(font
-					(size 1.27 1.27)
-				)
-				(justify right)
-			)
-		)
-	)
-	(global_label "O2_SENSOR_RX"
+	)
+	(hierarchical_label "O2_SENSOR_RX"
 		(shape output)
-		(at 186.69 118.11 180)
-		(fields_autoplaced yes)
+		(at 189.23 109.22 180)
 		(effects
 			(font
@@
 			(justify right)
 		)
-		(property "Intersheetrefs" "${INTERSHEET_REFS}"
-			(at 169.2511 118.11 0)
-			(hide yes)
-			(show_name no)
-			(do_not_autoplace no)
-			(effects
-				(font
-					(size 1.27 1.27)
-				)
-				(justify right)
-			)
-		)
-	)
+	)

Commit message: Updated board for layout! All footprints added
Parts:
- J7: footprint (none) -> Connector_Molex:Molex_Micro-Fit_3.0_43045-0400_2x02_P3.00mm_Horizontal; BOM Source (none) -> https://www.molex.com/en-us/products/part-detail/430450400; MPN (none) -> 0430450400; Manufacturer (none) -> Molex
Changed lines of the file:
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@@
 			)
 		)
-		(property "Footprint" ""
+		(property "Footprint" "Connector_Molex:Molex_Micro-Fit_3.0_43045-0400_2x02_P3.00mm_Horizontal"
 			(at 198.12 106.68 0)
 			(hide yes)
@@
 			(hide yes)
 			(show_name no)
+			(do_not_autoplace no)
+			(effects
+				(font
+					(size 1.27 1.27)
+				)
+			)
+		)
+		(property "MPN" "0430450400"
+			(at 0 0 0)
+			(hide yes)
+			(show_name no)
+			(do_not_autoplace no)
+			(effects
+				(font
+					(size 1.27 1.27)
+				)
+			)
+		)
+		(property "Manufacturer" "Molex"
+			(at 0 0 0)
+			(hide yes)
+			(show_name no)
+			(do_not_autoplace no)
+			(effects
+				(font
+					(size 1.27 1.27)
+				)
+			)
+		)
+		(property "BOM Source" "https://www.molex.com/en-us/products/part-detail/430450400"
+			(at 0 0 0)
+			(hide yes)
+			(show_name no)

Commit message: Let gpt6 astra have a go at routing. bad results.
Parts:
- U38: footprint Package_SO:Texas_HTSSOP-14-1EP_4.4x5mm_P0.65mm_EP3.4x5mm_Mask3.155x3.255mm_ThermalVias -> DIC_Board:TPS27S100_Thermal_Drill0p3
Changed lines of the file:
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@@
 			)
 		)
-		(property "Footprint" "Package_SO:Texas_HTSSOP-14-1EP_4.4x5mm_P0.65mm_EP3.4x5mm_Mask3.155x3.255mm_ThermalVias"
+		(property "Footprint" "DIC_Board:TPS27S100_Thermal_Drill0p3"
 			(at 134.62 101.6 0)
 			(hide yes)
