File: DIC_Board/5v.kicad_sch (KiCad schematic)
At the start: 12 parts, among them U12 TPSM53603RDAR

Commit message: Preliminary layout
Parts:
- TP24: footprint TestPoint:TestPoint_Plated_Hole_D2.0mm -> TestPoint:TestPoint_Pad_D1.0mm
Changed lines of the file:
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@@
 			)
 		)
-		(property "Footprint" "TestPoint:TestPoint_Plated_Hole_D2.0mm"
+		(property "Footprint" "TestPoint:TestPoint_Pad_D1.0mm"
 			(at 224.79 92.71 0)
 			(hide yes)
